File: Hardware/Crenshaw.sch (KiCad schematic (older format))
At the start: 18 parts, among them J1 Jumper_Voltage, J2 I2C, J3 I2C, P1 SSD1306_ribbon, U1 AP2112K-3.3

Commit message: SOD323 schottky switched to SOD123
Bigger means less heat issues
Parts:
- D1: footprint Diode_SMD:D_SOD-323 -> Diode_SMD:D_SOD-123
Changed lines of the file:
@@
 F 0 "D1" V 4700 2050 50  0000 C CNN
 F 1 "<.5Vf" V 4800 2050 50  0000 C CNN
-F 2 "Diode_SMD:D_SOD-323" V 4750 2200 50  0001 C CNN
+F 2 "Diode_SMD:D_SOD-123" V 4750 2200 50  0001 C CNN
 F 3 "" V 4750 2200 50  0000 C CNN
 	1    4750 2200
